File: UnOrthoDox 20 PCB/UnOrthoDox 20 PCB.kicad_sch (KiCad schematic)
At the start: 70 parts, among them SW1 SW_MX_HotSwap, SW10 SW_MX_HotSwap, SW11 SW_MX_HotSwap, SW12 SW_MX_HotSwap, SW13 SW_MX_HotSwap, SW14 SW_MX_HotSwap, SW15 SW_MX_HotSwap, SW16 SW_MX_HotSwap, SW17 SW_MX_HotSwap, SW18 SW_MX_HotSwap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

Commit message: Final tweaks 17/20 PCB
Parts:
- RGB1, RGB10, RGB11, RGB12, RGB13, RGB14, RGB15, RGB16, RGB17, RGB18, RGB19, RGB2, RGB20, RGB3, RGB4, RGB5, RGB6, RGB7, RGB8, RGB9: footprint Keyboard RGB:MX_SK6812MINI-E_REVERSIBLE -> Keyboard RGB:RGB_SK6812MINI-E
- RZ1: footprint Keyboard Controllers:RP2040-Zero_reverse_mount_flipped -> Keyboard Controllers:RP2040-Zero_reverse_mount_flipped_less_pins
- SW1, SW10, SW11, SW12, SW13, SW14, SW15, SW16, SW17, SW18, SW19, SW2, SW20, SW3, SW4, SW5, SW6, SW7, SW8, SW9: footprint Keyboard Switches:SW_MX_HotSwap_Reversible -> Keyboard Switches:SW_MX_HotSwap
