File: UnOrthoDox Rear/UnOrthoDox Rear.kicad_pcb (KiCad board)
At the start: 2 copper layers, 88.2 x 97.2 mm, 4 parts

Commit message: Reworked plates for release
Parts:
- moved H1 2.50 mm to (107.3, 32.6)
- moved H3 2.50 mm to (189.5, 32.6)
- moved H2 0.25 mm to (107.3, 126.6)
- moved H4 0.25 mm to (189.5, 126.6)
Other:
- board size 88.2 x 97.2 mm -> 88.2 x 100 mm
- board text added: "1. Determine the layout and orientation, and solder the hotswap sockets needed. - Keep in mind that sockets overlap on optional placements. - Do NOT attempt to solder all sockets! 2. Solder ALL diodes. (Place the line on the diode to the marking on PCB) 3. Solder level shifter for RGB. (SMD, optional if not using RGB) 4. Solder capacitors for Encoders. (unidirectional, optional if not using encod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"
- board text added: "UnOrthoDox Rear - v1.0.0"
- board text removed: "1. Solder ALL diodes. (Place the line on the diode to the marking on PCB) 2. Determine the layout and solder the hotswap sockets needed. - Keep in mind that sockets overlap on the optional placements. - Do NOT attempt to solder all sockets! 3. Solder reset switch, and optionally the powerswitch for a wireless build. 4. Solder capacitors for optional Encoders. (unidirectional) 5. Solder RGB LED's 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"
- board text removed: "UnOrthoDox 20 Rear - v1.0.0"

Commit message: Updated renders
Parts:
- added H1: Spacer_PCB, Keyboard_Plate:Spacer Plate hole, F.Cu at (143.8, 46.7)
- added H1: Spacer_PCB, Keyboard_Plate:Spacer Plate hole, F.Cu at (133.8, 46.7)
Changed lines of the file:
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@@
+    (pad "" np_thru_hole circle (at 0 0 90) (size 2.5 2.5) (drill 2.5) (layers "*.Cu" "*.Mask"))
+  )
+  (footprint "Keyboard_Plate:Spacer Plate hole" (layer "F.Cu")
+    (at 143.84 46.66 90)
+    (descr "Mounting Hole 2.5mm, no annular")
+    (tags "mounting hole 2.5mm no annular")
+    (property "Sheetfile" "UnOrthoDox 20 Rear.kicad_sch")
+    (property "Sheetname" "")
+    (attr exclude_from_pos_files)
+    (fp_text reference "H1" (at 0 -3.5 90) (layer "F.SilkS") hide
+        (effects (font (size 1 1) (thickness 0.15)))
+    )
+    (fp_text value "Spacer_PCB" (at 0 3.5 90) (layer "F.Fab") hide
+        (effects (font (size 1 1) (thickness 0.15)))
+    )
+    (fp_text user "${REFERENCE}" (at 0 0 90) (layer "F.Fab")
+        (effects (font (size 1 1) (thickness 0.15)))
+    )
+    (fp_circle (center 0 0) (end 2.5 0)
+      (stroke (width 0.15) (type solid)) (fill none) (layer "Cmts.User"))
+    (fp_circle (center 0 0) (end 2.75 0)
+      (stroke (width 0.05) (type solid)) (fill none) (layer "F.CrtYd"))
+    (pad "" np_thru_hole circle (at 0 0 90) (size 2.5 2.5) (drill 2.5) (layers "*.Cu" "*.Mask"))
+  )
+  (footprint "Keyboard_Plate:Spacer Plate hole" (layer "F.Cu")
+    (at 133.84 46.66 90)
+    (descr "Mounting Hole 2.5mm, no annular")
+    (tags "mounting hole 2.5mm no annular")
+    (property "Sheetfile" "UnOrthoDox 20 Rear.kicad_sch")
+    (property "Sheetname" "")
+    (attr exclude_from_pos_files)
+    (fp_text reference "H1" (at 0 -3.5 90) (layer "F.SilkS") hide
+        (effects (font (size 1 1) (thickness 0.15)))
+    )
+    (fp_text value "Spacer_PCB" (at 0 3.5 90) (layer "F.Fab") hide
+        (effects (font (size 1 1) (thickness 0.15)))
+    )
+    (fp_text user "${REFERENCE}" (at 0 0 90) (layer "F.Fab")
+        (effects (font (size 1 1) (thickness 0.15)))
+    )
+    (fp_circle (center 0 0) (end 2.5 0)
+      (stroke (width 0.15) (type solid)) (fill none) (layer "Cmts.User"))
+    (fp_circle (center 0 0) (end 2.75 0)
+      (stroke (width 0.05) (type solid)) (fill none) (layer "F.CrtYd"))
     (pad "" np_thru_hole circle (at 0 0 90) (size 2.5 2.5) (drill 2.5) (layers "*.Cu" "*.Mask"))
   )
@@
   (gr_arc (start 189.46 29.64) (mid 191.58132 30.51868) (end 192.46 32.64)
     (stroke (width 0.1) (type solid)) (layer "Edge.Cuts"))
-  (gr_text "1. Determine the layout and orientation, and solder the hotswap sockets needed.\n   - Keep in mind that sockets overlap on optional placements.\n   - Do NOT attempt to solder all sockets!\n\n2. Solder ALL diodes. (Place the line on the diode to the marking on PCB)\n\n3. Solder level shifter for RGB. (SMD, optional if not using RGB)\n\n4. Solder capacitors for Encoders. (unidirectional, optional if not using encoders)\n\n5. Solder RGB LED's in place. (Orient notched leg to marking)\n   - Solder the RGB ONLY for the switch positions used!\n   - RGB's for optional layouts are in paralell and will not work if all are soldered!\n\n6. Solder controller/socket for controller. \n   - Cut socket strip to use only the marked pins. \n   - Solder pins only in the used holes!\n   - Diode legs are preferred over square pin strip!\n   - Controller is oriented with reset buttosn facing out (reversed on 17 Southpaw).\n\n7. Solder optional Encoders in place.\n\n8. Assemble & Enjoy!" (at 116.93 78.75) (layer "F.SilkS")
+  (gr_text "1. Determine the layout and orientation, and solder the hotswap sockets needed.\n   - Keep in mind that sockets overlap on optional placements.\n   - Do NOT attempt to solder all sockets!\n\n2. Solder ALL diodes. (Place the line on the diode to the marking on PCB)\n\n3. Solder level shifter for RGB. (SMD, optional if not using RGB)\n\n4. Solder capacitors for Encoders. (unidirectional, optional if not using encoders)\n\n5. Solder RGB LED's in place. (Orient notched leg to marking)\n   - Solder the RGB ONLY for the switch positions used!\n   - RGB's for optional layouts are in paralell and will not work if all are soldered!\n\n6. Solder controller/socket for controller. \n   - Cut socket strip to use only the marked pins. \n   - Solder pins only in the used holes!\n   - Diode legs are preferred over square pin strip!\n   - Controller is oriented with reset buttosn facing out (reversed on 17 Southpaw).\n\n7. Solder optional Encoders in place.\n\n8. Assemble & Enjoy!" (at 116.93 83.75) (layer "F.SilkS")
     (effects (font (size 1 1) (thickness 0.15)) (justify left))
   )
-  (gr_text "JLCJLCJLCJLC" (at 165.2 49.13) (layer "F.SilkS")
+  (gr_text "JLCJLCJLCJLC" (at 165.2 54.13) (layer "F.SilkS")
     (effects (font (size 1 1) (thickness 0.15)))
   )
-  (gr_text "UnOrthoDox Rear - v1.0.0" (at 138.66 49.13) (layer "F.SilkS")
+  (gr_text "UnOrthoDox Rear - v1.0.0" (at 138.66 54.13) (layer "F.SilkS")
     (effects (font (size 1 1) (thickness 0.15)))
   )
